File: test1.kicad_pcb (KiCad board)
At the start: 2 copper layers, 7 parts, among them J1 MLX, J2 ON/OFF, J3 BNO, J4 tp4056, J5 BNO, J6 soket, U1 XIAO-ESP32-C3-SMD

Commit message: upd sedikit
Parts:
- moved U1 26.7 mm to (86.6, 57.7), turned to -90 degrees
- moved J6 22.9 mm to (80.0, 68.7)
- moved J2 22.0 mm to (69.5, 65.2)
- moved J4 19.9 mm to (62.0, 62.0)
Routing:
- net /OUT-: track 158.3 -> 123.0 mm
- net Net-(J1-Pin_3): track 86.1 -> 58.2 mm
- net Net-(J1-Pin_4): track 81.8 -> 55.0 mm
- net /sda/dx: track 58.0 -> 84.5 mm
- net Net-(J2-Pin_2): track 69.9 -> 44.8 mm
- net /B+: track 32.0 -> 20.9 mm
- net /OUT+: track 14.5 -> 8.84 mm
- net unconnected-(U1-GPIO10_D10_MOSI-Pad11): track 0.00 -> 1.46 mm
- net /B-: track 28.0 -> 28.9 mm

Commit message: upd sedikitlagi - beresin footprint sama stl
Other:
- board outline added: 70 x 32 mm
Changed lines of the file:
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@@
 	)
 	(gr_rect
-		(start 40.1723 47.705164)
-		(end 110.1723 77.705164)
+		(start 40 45)
+		(end 110 80)
 		(stroke
 			(width 0.2)
@@
 		(layer "F.Cu")
 	)
+	(gr_rect
+		(start 40 48)
+		(end 110 80)
+		(stroke
+			(width 0.1)
+			(type solid)
+		)
+		(fill no)
+		(layer "Edge.Cuts")
+	)
 	(segment
